File: KiCad/K-Pillar.kicad_pcb (KiCad board)
At the start: 2 copper layers, 45 x 50 mm, 14 parts, among them J1 I2COut, J2 Keypad, J3 Relay, M1 Pump, M2 Pump, M3 Pump, Q1 IRLZ44N, Q2 IRLZ44N, Q3 IRLZ44N

Commit message: board v2
Parts:
- added J4: RTC, Connector_PinHeader_2.54mm:PinHeader_1x07_P2.54mm_Vertical, F.Cu at (27.5, 27.4)
- added R1: 4k7, Resistor_SMD:R_0805_2012Metric_Pad1.20x1.40mm_HandSolder, B.Cu at (43.2, 36.5)
- added R2: 10k, Resistor_SMD:R_0805_2012Metric_Pad1.20x1.40mm_HandSolder, B.Cu at (43.0, 58.0)
- added REF**: jakubkivi.github.io, SVGs:jakubkivi.github.io, F.Cu at (59.8, 64.9)
- moved J2 12.5 mm to (27.5, 48.4)
- moved Q1 1.00 mm to (52.0, 66.4)
- moved Q2 1.00 mm to (52.0, 59.4)
- moved Q3 1.00 mm to (52.0, 52.4)
Connections:
- net Net-(A1-A4) renamed RTC_SDA
- net Net-(A1-A5) renamed RTC_SCL
- A1 pad 12: unconnected-(A1-D9-Pad12) -> PUMP3
- A1 pad 13: unconnected-(A1-D10-Pad13) -> PUMP2
- A1 pad 14: unconnected-(A1-D11-Pad14) -> PUMP1
- A1 pad 15: unconnected-(A1-D12-Pad15) -> Net-(A1-D12)
- A1 pad 17: unconnected-(A1-3V3-Pad17) -> Net-(A1-3V3)
- A1 pad 18: unconnected-(A1-AREF-Pad18) -> Net-(A1-AREF)
- A1 pad 19: PUMP1 -> unconnected-(A1-A0-Pad19)
- A1 pad 20: PUMP2 -> unconnected-(A1-A1-Pad20)
- A1 pad 21: PUMP3 -> unconnected-(A1-A2-Pad21)
- A1 pad 25: unconnected-(A1-A6-Pad25) -> RTC_DS
- A1 pad 26: unconnected-(A1-A7-Pad26) -> RTC_BAT
- A1 pad 5: Net-(A1-D2) -> RTC_SQ
- J2 pad 1: Net-(A1-D2) -> Net-(A1-D3)
- J2 pad 2: Net-(A1-D3) -> Net-(A1-D4)
- J2 pad 3: Net-(A1-D4) -> Net-(A1-D5)
- J2 pad 4: Net-(A1-D5) -> Net-(A1-D6)
- J2 pad 5: Net-(A1-D6) -> Net-(A1-D7)
- J2 pad 6: Net-(A1-D7) -> Net-(A1-D8)
- J2 pad 7: Net-(A1-D8) -> Net-(A1-D12)
Routing:
- net PUMP3: track 7.74 -> 34.5 mm
- net +5V: track 39.7 -> 66.2 mm, vias 1 -> 2
- net RTC_SDA: track 5.91 -> 31.9 mm, vias 0 -> 1
- net RTC_DS: track 0.00 -> 25.5 mm, vias 0 -> 1
- net RTC_BAT: track 0.00 -> 23.0 mm
- net RTC_SCL: track 5.91 -> 26.8 mm
- net PUMP2: track 11.9 -> 27.4 mm
- net RTC_SQ: track 0.00 -> 9.61 mm
- net Net-(A1-D4): track 3.57 -> 12.7 mm
- net Net-(A1-D6): track 3.57 -> 12.5 mm
- net Net-(A1-D7): track 3.57 -> 12.2 mm
- net Net-(A1-D5): track 3.57 -> 11.7 mm
- net PUMP1: track 15.5 -> 23.6 mm
- net Net-(A1-D3): track 3.57 -> 11.5 mm
- net Net-(A1-D8): track 3.57 -> 11.5 mm
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Other:
- board text added: "K-Pillar"
- board text added: "v2"
